File: sondeSide.brd (EAGLE design)
At the start: 66.8 x 32 mm, 32 parts

Commit message: Finally ready to send with holes and everything
Routing:
- net 3.3V: track 63.2 -> 64.5 mm
Changed lines of the file:
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@@
 <layer number="43" name="vRestrict" color="2" fill="10" visible="yes" active="yes"/>
 <layer number="44" name="Drills" color="7" fill="1" visible="no" active="yes"/>
-<layer number="45" name="Holes" color="7" fill="1" visible="no" active="yes"/>
+<layer number="45" name="Holes" color="7" fill="1" visible="yes" active="yes"/>
 <layer number="46" name="Milling" color="3" fill="1" visible="no" active="yes"/>
 <layer number="47" name="Measures" color="7" fill="1" visible="no" active="yes"/>
@@
 <wire x1="55.626" y1="13.208" x2="55.626" y2="27.686" width="0.127" layer="21"/>
 <wire x1="55.626" y1="27.686" x2="55.88" y2="27.686" width="0.127" layer="21"/>
+<hole x="3.175" y="19.685" drill="2.54"/>
+<hole x="24.384" y="9.0678" drill="4.318"/>
+<hole x="3.175" y="3.175" drill="2.54"/>
+<wire x1="1.143" y1="22.86" x2="36.322" y2="22.86" width="0.025" layer="49"/>
 </plain>
 <attributes>
@@
 <wire x1="41.402" y1="12.446" x2="41.402" y2="11.557" width="0.8128" layer="16"/>
 <wire x1="41.402" y1="11.557" x2="40.767" y2="10.922" width="0.8128" layer="16"/>
-<wire x1="41.402" y1="14.986" x2="27.686" y2="14.986" width="1.524" layer="16"/>
-<wire x1="27.686" y1="14.986" x2="22.352" y2="20.32" width="1.524" layer="16"/>
-<wire x1="22.352" y1="20.32" x2="22.352" y2="23.368" width="1.524" layer="16"/>
+<wire x1="23.368" y1="24.638" x2="23.368" y2="19.304" width="1.524" layer="16"/>
 <wire x1="10.16" y1="28.448" x2="10.16" y2="29.972" width="1.524" layer="16"/>
-<via x="22.352" y="23.368" extent="1-16" drill="0.35"/>
-<wire x1="22.352" y1="23.368" x2="19.05" y2="26.67" width="1.524" layer="1"/>
-<via x="19.05" y="26.67" extent="1-16" drill="0.35"/>
-<wire x1="11.938" y1="26.67" x2="10.16" y2="28.448" width="1.524" layer="16"/>
-<wire x1="19.05" y1="26.67" x2="11.938" y2="26.67" width="1.524" layer="16"/>
-<wire x1="41.402" y1="14.986" x2="43.688" y2="24.892" width="0" layer="19" extent="16-16"/>
+<via x="23.368" y="24.638" extent="1-16" drill="0.35"/>
+<wire x1="23.368" y1="24.638" x2="20.32" y2="27.686" width="1.524" layer="1"/>
+<via x="20.32" y="27.686" extent="1-16" drill="0.35"/>
+<wire x1="10.922" y1="27.686" x2="10.16" y2="28.448" width="1.524" layer="16"/>
+<wire x1="20.32" y1="27.686" x2="10.922" y2="27.686" width="1.524" layer="16"/>
+<wire x1="23.368" y1="19.304" x2="25.4" y2="17.272" width="1.524" layer="16"/>
+<wire x1="39.37" y1="14.986" x2="41.402" y2="14.986" width="1.524" layer="16"/>
+<wire x1="25.4" y1="17.272" x2="37.084" y2="17.272" width="1.524" layer="16"/>
+<wire x1="37.084" y1="17.272" x2="39.37" y2="14.986" width="1.524" layer="16"/>
+<wire x1="37.084" y1="17.272" x2="36.322" y2="24.892" width="0" layer="19" extent="16-16"/>
 </signal>
 <signal name="GND">
@@
 <wire x1="35.56" y1="29.972" x2="35.433" y2="29.972" width="0.1524" layer="16"/>
 <wire x1="23.114" y1="28.067" x2="18.9564" y2="23.9094" width="0.1524" layer="16"/>
-<wire x1="18.9564" y1="19.3976" x2="29.972" y2="8.382" width="0.1524" layer="16"/>
-<wire x1="29.972" y1="8.382" x2="40.767" y2="8.382" width="0.1524" layer="16"/>
-<wire x1="18.9564" y1="23.9094" x2="18.9564" y2="19.3976" width="0.1524" layer="16"/>
+<wire x1="18.9564" y1="19.3976" x2="18.9564" y2="23.9094" width="0.1524" layer="16"/>
+<wire x1="40.767" y1="8.382" x2="37.338" y2="8.382" width="0.1524" layer="16"/>
+<wire x1="23.876" y1="14.478" x2="18.9564" y2="19.3976" width="0.1524" layer="16"/>
+<wire x1="37.338" y1="8.382" x2="31.242" y2="14.478" width="0.1524" layer="16"/>
+<wire x1="31.242" y1="14.478" x2="23.876" y2="14.478" width="0.1524" layer="16"/>
 </signal>
 <signal name="TX2">
@@
 <wire x1="31.496" y1="28.448" x2="28.448" y2="28.448" width="0.1524" layer="16"/>
 <wire x1="28.448" y1="28.448" x2="28.194" y2="28.448" width="0.1524" layer="16"/>
-<wire x1="18.6516" y1="24.03565625" x2="18.6516" y2="19.27134375" width="0.1524" layer="16"/>
-<wire x1="18.6516" y1="19.27134375" x2="29.84574375" y2="8.0772" width="0.1524" layer="16"/>
+<wire x1="18.6516" y1="24.03565625" x2="18.6516" y2="19.304" width="0.1524" layer="16"/>
+<wire x1="18.6516" y1="19.304" x2="18.6516" y2="19.27134375" width="0.1524" layer="16"/>
 <wire x1="28.448" y1="28.448" x2="23.06394375" y2="28.448" width="0.1524" layer="16"/>
 <wire x1="23.06394375" y1="28.448" x2="18.6516" y2="24.03565625" width="0.1524" layer="16"/>
 <wire x1="38.5318" y1="8.0772" x2="40.767" y2="5.842" width="0.1524" layer="16"/>
-<wire x1="29.84574375" y1="8.0772" x2="38.5318" y2="8.0772" width="0.1524" layer="16"/>
+<wire x1="18.6516" y1="19.304" x2="18.6516" y2="19.27134375" width="0.1524" layer="16"/>
+<wire x1="18.6516" y1="19.27134375" x2="23.74974375" y2="14.1732" width="0.1524" layer="16"/>
+<wire x1="31.11574375" y1="14.1732" x2="37.21174375" y2="8.0772" width="0.1524" layer="16"/>
+<wire x1="37.21174375" y1="8.0772" x2="38.5318" y2="8.0772" width="0.1524" layer="16"/>
+<wire x1="23.74974375" y1="14.1732" x2="31.11574375" y2="14.1732" width="0.1524" layer="16"/>
 </signal>
 <signal name="RX3">
@@
 <wire x1="40.64" y1="29.972" x2="37.846" y2="27.178" width="0.1524" layer="16"/>
 <wire x1="23.876" y1="27.178" x2="20.193" y2="23.495" width="0.1524" layer="16"/>
-<wire x1="20.193" y1="23.495" x2="20.193" y2="19.685" width="0.1524" layer="16"/>
+<wire x1="20.193" y1="23.495" x2="20.193" y2="19.812" width="0.1524" layer="16"/>
+<wire x1="20.193" y1="19.812" x2="20.193" y2="19.685" width="0.1524" layer="16"/>
 <wire x1="37.846" y1="27.178" x2="23.876" y2="27.178" width="0.1524" layer="16"/>
-<wire x1="20.193" y1="19.685" x2="30.099" y2="9.779" width="0.1524" layer="16"/>
-<wire x1="30.099" y1="9.779" x2="43.307" y2="9.779" width="0.1524" layer="16"/>
 <wire x1="43.307" y1="9.779" x2="46.228" y2="6.858" width="0.1524" layer="16"/>
 <wire x1="46.228" y1="3.048" x2="46.99" y2="2.286" width="0.1524" layer="16"/>
@@
 <wire x1="60.198" y1="9.398" x2="61.976" y2="7.62" width="0.1524" layer="16"/>
 <wire x1="61.976" y1="7.62" x2="61.976" y2="7.493" width="0.1524" layer="16"/>
+<wire x1="37.719" y1="9.779" x2="43.307" y2="9.779" width="0.1524" layer="16"/>
+<wire x1="34.29" y1="13.208" x2="34.544" y2="12.954" width="0.1524" layer="16"/>
+<wire x1="34.544" y1="12.954" x2="37.719" y2="9.779" width="0.1524" layer="16"/>
+<wire x1="20.193" y1="19.685" x2="24.384" y2="15.494" width="0.1524" layer="16"/>
+<wire x1="32.004" y1="15.494" x2="34.544" y2="12.954" width="0.1524" layer="16"/>
+<wire x1="24.384" y1="15.494" x2="32.004" y2="15.494" width="0.1524" layer="16"/>
 </signal>
 <signal name="TX3">
@@
 <wire x1="23.6982" y1="27.5082" x2="19.812" y2="23.622" width="0.1524" layer="16"/>
 <wire x1="19.812" y1="23.622" x2="19.812" y2="19.558" width="0.1524" layer="16"/>
-<wire x1="19.812" y1="19.558" x2="29.972" y2="9.398" width="0.1524" layer="16"/>
-<wire x1="29.972" y1="9.398" x2="43.18" y2="9.398" width="0.1524" layer="16"/>
 <wire x1="43.18" y1="9.398" x2="45.9232" y2="6.6548" width="0.1524" layer="16"/>
 <wire x1="45.9232" y1="2.92174375" x2="46.86374375" y2="1.9812" width="0.1524" layer="16"/>
@@
 <wire x1="46.86374375" y1="1.9812" x2="54.48225625" y2="1.9812" width="0.1524" layer="16"/>
 <wire x1="30.988" y1="27.5082" x2="23.6982" y2="27.5082" width="0.1524" layer="16"/>
+<wire x1="37.66894375" y1="9.398" x2="43.18" y2="9.398" width="0.1524" layer="16"/>
+<wire x1="19.812" y1="19.558" x2="24.1808" y2="15.1892" width="0.1524" layer="16"/>
+<wire x1="24.1808" y1="15.1892" x2="31.87774375" y2="15.1892" width="0.1524" layer="16"/>
+<wire x1="31.87774375" y1="15.1892" x2="37.66894375" y2="9.398" width="0.1524" layer="16"/>
 </signal>
 <signal name="5V">
