File: sondeSide.sch (EAGLE design)
At the start: 41 parts

Commit message: Board is good to go
Parts:
- R3: value (none) -> 370Ω
Changed lines of the file:
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@@
 <part name="JP32" library="pinhead" library_urn="urn:adsk.eagle:library:325" deviceset="PINHD-1X1" device="" package3d_urn="urn:adsk.eagle:package:22485/2"/>
 <part name="OK1" library="optocoupler" library_urn="urn:adsk.eagle:library:320" deviceset="H11L*M" device="T" package3d_urn="urn:adsk.eagle:package:21968/1" technology="2"/>
-<part name="R3" library="rcl" library_urn="urn:adsk.eagle:library:334" deviceset="R-US_" device="0204/7" package3d_urn="urn:adsk.eagle:package:23498/1"/>
+<part name="R3" library="rcl" library_urn="urn:adsk.eagle:library:334" deviceset="R-US_" device="0204/7" package3d_urn="urn:adsk.eagle:package:23498/1" value="370Ω"/>
 </parts>
 <sheets>

Commit message: Last push before switching to live-switch SSR
Parts:
- added JP25: (no value), pinhead:PINHD-1X2
Connections:
- net GND: now also JP25.1
- net GND_PLANE: now also JP25.2
Other:
- note added: "Switch"
Changed lines of the file:
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@@
 <part name="OK1" library="optocoupler" library_urn="urn:adsk.eagle:library:320" deviceset="H11L*M" device="T" package3d_urn="urn:adsk.eagle:package:21968/1" technology="2"/>
 <part name="R3" library="rcl" library_urn="urn:adsk.eagle:library:334" deviceset="R-US_" device="0204/7" package3d_urn="urn:adsk.eagle:package:23498/1" value="370Ω"/>
+<part name="JP25" library="pinhead" library_urn="urn:adsk.eagle:library:325" deviceset="PINHD-1X2" device="" package3d_urn="urn:adsk.eagle:package:22435/2"/>
 </parts>
 <sheets>
@@
 <text x="0" y="-10.16" size="1.778" layer="91">"GND" is only connected to ground
 when the switch is closed</text>
+<text x="12.7" y="63.5" size="1.778" layer="91">Switch</text>
 </plain>
 <instances>
@@
 <instance part="OK1" gate="G$1" x="-12.7" y="-17.78"/>
 <instance part="R3" gate="G$1" x="-33.02" y="-15.24" rot="R180"/>
+<instance part="JP25" gate="G$1" x="17.78" y="53.34"/>
 </instances>
 <busses>
@@
 <wire x1="-2.54" y1="-15.24" x2="0" y2="-15.24" width="0.1524" layer="91"/>
 <label x="0" y="-15.24" size="1.778" layer="95"/>
+</segment>
+<segment>
+<pinref part="JP25" gate="G$1" pin="1"/>
+<wire x1="15.24" y1="55.88" x2="7.62" y2="55.88" width="0.1524" layer="91"/>
+<label x="7.62" y="55.88" size="1.778" layer="95" rot="R180"/>
 </segment>
 </net>
@@
 <wire x1="66.04" y1="63.5" x2="66.04" y2="68.58" width="0.1524" layer="91"/>
 </segment>
-</net>
+<segment>
+<pinref part="JP25" gate="G$1" pin="2"/>
+<wire x1="15.24" y1="53.34" x2="7.62" y2="53.34" width="0.1524" layer="91"/>
+<label x="7.62" y="53.34" size="1.778" layer="95" rot="R180"/>
+</segment>
+</net>

Commit message: Electrically ready to go
Parts:
- JP25: device pinhead:PINHD-1X2 -> con-lstb:MA03-1
- R3: device rcl:R-US_0204/7 -> rcl:R-US_0204/2V
Connections:
- removed net GND_PLANE: JP25.2, JP26.1, OK1.C, OK1.GND, PWRBOOST-1.S
- new net 5V_TO_SMPS: JP25.2, OK1.GND, STEP-DOWN-3.S, STEP-UP-1.S
- net 5V: now also JP25.1, OK1.OUT, OK1.VCC; no longer STEP-DOWN-3.S, STEP-UP-1.S
- net GND: now also JP26.1, OK1.C, PWRBOOST-1.S; no longer JP25.1, OK1.OUT, OK1.VCC
Other:
- note removed: ""GND" is only connected to ground when the switch is closed"
Changed lines of the file:
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@@
 <part name="JP22" library="pinhead" library_urn="urn:adsk.eagle:library:325" deviceset="PINHD-1X1" device="" package3d_urn="urn:adsk.eagle:package:22485/2"/>
 <part name="JP23" library="pinhead" library_urn="urn:adsk.eagle:library:325" deviceset="PINHD-1X1" device="" package3d_urn="urn:adsk.eagle:package:22485/2"/>
-<part name="JP24" library="pinhead" library_urn="urn:adsk.eagle:library:325" deviceset="PINHD-1X1" device="" package3d_urn="urn:adsk.eagle:package:22485/2"/>
 <part name="STEP-DOWN" library="con-molex" library_urn="urn:adsk.eagle:library:165" deviceset="22-23-2041" device=""/>
 <part name="PWRBOOST" library="con-molex" library_urn="urn:adsk.eagle:library:165" deviceset="22-23-2021" device=""/>
@@
 <part name="JP32" library="pinhead" library_urn="urn:adsk.eagle:library:325" deviceset="PINHD-1X1" device="" package3d_urn="urn:adsk.eagle:package:22485/2"/>
 <part name="OK1" library="optocoupler" library_urn="urn:adsk.eagle:library:320" deviceset="H11L*M" device="T" package3d_urn="urn:adsk.eagle:package:21968/1" technology="2"/>
-<part name="R3" library="rcl" library_urn="urn:adsk.eagle:library:334" deviceset="R-US_" device="0204/7" package3d_urn="urn:adsk.eagle:package:23498/1" value="370Ω"/>
-<part name="JP25" library="pinhead" library_urn="urn:adsk.eagle:library:325" deviceset="PINHD-1X2" device="" package3d_urn="urn:adsk.eagle:package:22435/2"/>
+<part name="R3" library="rcl" library_urn="urn:adsk.eagle:library:334" deviceset="R-US_" device="0204/2V" package3d_urn="urn:adsk.eagle:package:23495/1" value="370Ω"/>
+<part name="JP25" library="con-lstb" library_urn="urn:adsk.eagle:library:162" deviceset="MA03-1" device="" package3d_urn="urn:adsk.eagle:package:8339/1"/>
+<part name="JP24" library="pinhead" library_urn="urn:adsk.eagle:library:325" deviceset="PINHD-1X1" device="" package3d_urn="urn:adsk.eagle:package:22485/2"/>
 </parts>
 <sheets>
@@
 <text x="-58.42" y="76.2" size="1.778" layer="91">Teensy</text>
 <text x="-60.96" y="-2.54" size="1.778" layer="91">Receiver</text>
-<text x="0" y="-10.16" size="1.778" layer="91">"GND" is only connected to ground
-when the switch is closed</text>
 <text x="12.7" y="63.5" size="1.778" layer="91">Switch</text>
 </plain>
@@
 <instance part="JP22" gate="G$1" x="-58.42" y="17.78" rot="R180"/>
 <instance part="JP23" gate="G$1" x="-58.42" y="15.24" rot="R180"/>
-<instance part="JP24" gate="G$1" x="-58.42" y="12.7" rot="R180"/>
 <instance part="STEP-DOWN" gate="-1" x="68.58" y="53.34"/>
 <instance part="STEP-DOWN" gate="-2" x="68.58" y="50.8"/>
@@
 <instance part="OK1" gate="G$1" x="-12.7" y="-17.78"/>
 <instance part="R3" gate="G$1" x="-33.02" y="-15.24" rot="R180"/>
-<instance part="JP25" gate="G$1" x="17.78" y="53.34"/>
+<instance part="JP25" gate="G$1" x="17.78" y="53.34" rot="R180"/>
+<instance part="JP24" gate="G$1" x="-58.42" y="12.7" rot="R180"/>
 </instances>
 <busses>
@@
 </segment>
 <segment>
-<pinref part="OK1" gate="G$1" pin="OUT"/>
-<wire x1="-2.54" y1="-17.78" x2="0" y2="-17.78" width="0.1524" layer="91"/>
-<label x="0" y="-17.78" size="1.778" layer="95"/>
-</segment>
-<segment>
-<pinref part="OK1" gate="G$1" pin="VCC"/>
-<wire x1="-2.54" y1="-15.24" x2="0" y2="-15.24" width="0.1524" layer="91"/>
-<label x="0" y="-15.24" size="1.778" layer="95"/>
-</segment>
-<segment>
-<pinref part="JP25" gate="G$1" pin="1"/>
-<wire x1="15.24" y1="55.88" x2="7.62" y2="55.88" width="0.1524" layer="91"/>
-<label x="7.62" y="55.88" size="1.778" layer="95" rot="R180"/>
+<wire x1="-58.42" y1="-7.62" x2="-43.18" y2="-7.62" width="0.1524" layer="91"/>
+<wire x1="-58.42" y1="-7.62" x2="-63.5" y2="-7.62" width="0.1524" layer="91"/>
+<pinref part="JP26" gate="G$1" pin="1"/>
+<wire x1="-63.5" y1="-7.62" x2="-66.04" y2="-7.62" width="0.1524" layer="91"/>
+<junction x="-63.5" y="-7.62"/>
+<label x="-43.18" y="-7.62" size="1.778" layer="95"/>
+</segment>
+<segment>
+<pinref part="OK1" gate="G$1" pin="C"/>
+<wire x1="-22.86" y1="-20.32" x2="-25.4" y2="-20.32" width="0.1524" layer="91"/>
+<wire x1="-25.4" y1="-20.32" x2="-25.4" y2="-25.4" width="0.1524" layer="91"/>
+<label x="-25.4" y="-25.4" size="1.778" layer="95" rot="R180"/>
+</segment>
+<segment>
+<wire x1="66.04" y1="68.58" x2="60.96" y2="68.58" width="0.1524" layer="91"/>
+<pinref part="PWRBOOST" gate="-1" pin="S"/>
+<wire x1="68.58" y1="63.5" x2="66.04" y2="63.5" width="0.1524" layer="91"/>
+<wire x1="66.04" y1="63.5" x2="66.04" y2="68.58" width="0.1524" layer="91"/>
+<label x="60.96" y="68.58" size="1.778" layer="95" rot="R180"/>
 </segment>
 </net>
@@
 </segment>
 <segment>
-<pinref part="STEP-UP" gate="-1" pin="S"/>
-<wire x1="66.04" y1="30.48" x2="60.96" y2="30.48" width="0.1524" layer="91"/>
-<label x="60.96" y="30.48" size="1.778" layer="95" rot="R180"/>
-</segment>
-<segment>
-<pinref part="STEP-DOWN" gate="-3" pin="S"/>
-<wire x1="66.04" y1="48.26" x2="60.96" y2="48.26" width="0.1524" layer="91"/>
-<label x="60.96" y="48.26" size="1.778" layer="95" rot="R180"/>
-</segment>
-<segment>
 <wire x1="-66.04" y1="-10.16" x2="-63.5" y2="-10.16" width="0.1524" layer="91"/>
 <label x="-43.18" y="-10.16" size="1.778" layer="95"/>
@@
 <wire x1="-63.5" y1="-10.16" x2="-43.18" y2="-10.16" width="0.1524" layer="91"/>
 <junction x="-63.5" y="-10.16"/>
+</segment>
+<segment>
+<pinref part="OK1" gate="G$1" pin="VCC"/>
+<wire x1="-2.54" y1="-15.24" x2="0" y2="-15.24" width="0.1524" layer="91"/>
+<label x="0" y="-15.24" size="1.778" layer="95"/>
+</segment>
+<segment>
+<pinref part="OK1" gate="G$1" pin="OUT"/>
+<wire x1="-2.54" y1="-17.78" x2="0" y2="-17.78" width="0.1524" layer="91"/>
+<label x="0" y="-17.78" size="1.778" layer="95"/>
+</segment>
+<segment>
+<pinref part="JP25" gate="G$1" pin="1"/>
+<wire x1="10.16" y1="55.88" x2="7.62" y2="55.88" width="0.1524" layer="91"/>
+<label x="7.62" y="55.88" size="1.778" layer="95" rot="R180"/>
 </segment>
 </net>
@@
 </segment>
 </net>
-<net name="GND_PLANE" class="0">
-<segment>
-<wire x1="-58.42" y1="-7.62" x2="-43.18" y2="-7.62" width="0.1524" layer="91"/>
-<label x="-43.18" y="-7.62" size="1.778" layer="95"/>
-<wire x1="-58.42" y1="-7.62" x2="-63.5" y2="-7.62" width="0.1524" layer="91"/>
-<pinref part="JP26" gate="G$1" pin="1"/>
-<wire x1="-63.5" y1="-7.62" x2="-66.04" y2="-7.62" width="0.1524" layer="91"/>
-<junction x="-63.5" y="-7.62"/>
-</segment>
-<segment>
-<pinref part="OK1" gate="G$1" pin="C"/>
-<wire x1="-22.86" y1="-20.32" x2="-25.4" y2="-20.32" width="0.1524" layer="91"/>
-<wire x1="-25.4" y1="-20.32" x2="-25.4" y2="-25.4" width="0.1524" layer="91"/>
-<label x="-25.4" y="-25.4" size="1.778" layer="95" rot="R180"/>
-</segment>
-<segment>
-<pinref part="OK1" gate="G$1" pin="GND"/>
-<wire x1="-2.54" y1="-20.32" x2="0" y2="-20.32" width="0.1524" layer="91"/>
-<wire x1="0" y1="-20.32" x2="0" y2="-25.4" width="0.1524" layer="91"/>
-<label x="0" y="-25.4" size="1.778" layer="95"/>
-</segment>
-<segment>
-<wire x1="66.04" y1="68.58" x2="60.96" y2="68.58" width="0.1524" layer="91"/>
-<label x="60.96" y="68.58" size="1.778" layer="95" rot="R180"/>
-<pinref part="PWRBOOST" gate="-1" pin="S"/>
-<wire x1="68.58" y1="63.5" x2="66.04" y2="63.5" width="0.1524" layer="91"/>
-<wire x1="66.04" y1="63.5" x2="66.04" y2="68.58" width="0.1524" layer="91"/>
-</segment>
-<segment>
-<pinref part="JP25" gate="G$1" pin="2"/>
-<wire x1="15.24" y1="53.34" x2="7.62" y2="53.34" width="0.1524" layer="91"/>
-<label x="7.62" y="53.34" size="1.778" layer="95" rot="R180"/>
-</segment>
-</net>
 <net name="D0" class="0">
 <segment>
@@
 <wire x1="-63.5" y1="-22.86" x2="-66.04" y2="-22.86" width="0.1524" layer="91"/>
 <junction x="-63.5" y="-22.86"/>
+</segment>
+</net>
+<net name="5V_TO_SMPS" class="0">
+<segment>
+<pinref part="OK1" gate="G$1" pin="GND"/>
+<wire x1="-2.54" y1="-20.32" x2="0" y2="-20.32" width="0.1524" layer="91"/>
+<wire x1="0" y1="-20.32" x2="0" y2="-25.4" width="0.1524" layer="91"/>
+<label x="0" y="-25.4" size="1.778" layer="95"/>
+</segment>
+<segment>
+<pinref part="STEP-DOWN" gate="-3" pin="S"/>
+<wire x1="66.04" y1="48.26" x2="60.96" y2="48.26" width="0.1524" layer="91"/>
+<label x="60.96" y="48.26" size="1.778" layer="95" rot="R180"/>
+</segment>
+<segment>
+<pinref part="STEP-UP" gate="-1" pin="S"/>
+<wire x1="66.04" y1="30.48" x2="60.96" y2="30.48" width="0.1524" layer="91"/>
+<label x="60.96" y="30.48" size="1.778" layer="95" rot="R180"/>
+</segment>
+<segment>
+<pinref part="JP25" gate="G$1" pin="2"/>
+<wire x1="10.16" y1="53.34" x2="7.62" y2="53.34" width="0.1524" layer="91"/>
+<label x="7.62" y="53.34" size="1.778" layer="95" rot="R180"/>
 </segment>
 </net>
@@
 </drawing>
 <compatibility>
-<note version="6.3" minversion="6.2.2" severity="warning">
-Since Version 6.2.2 text objects can contain more than one line,
-which will not be processed correctly with this version.
-</note>
 <note version="8.2" severity="warning">
 Since Version 8.2, EAGLE supports online libraries. The ids
